File: deck_v3/napari-pcb/napari-pcb.kicad_pcb (KiCad board)
At the start: 2 copper layers, 142 x 78 mm, 62 parts, among them J1 USB_C_Receptacle_USB2.0_16P, J11 DNP, J12 CONN_PB_SIG, J13 CONN_PB_GND, J14 CONN_PB_VDD, J17 CONN_PD_SIG, J18 CONN_GND, J19 CONN_VDD, J2 Cirque, J20 CONN_PD_GND, J21 CONN_PD_VDD, J3 Cirque, J4 CONN_ENC_DEV, J5 Cirque A MCU, J6 CONN_ENC_MCU, J7 Cirque B MCU, J8 CONN_PA_SIG, J9 CONN_PA_GND, SW1 SW_Push, SW10 SW_Push, SW11 SW_Push, SW12 SW_Push, SW13 SW_Push, SW14 SW_Push, SW15 SW_Push, SW16 SW_Push, SW2 SW_Push, SW3 SW_Push, SW4 SW_Push, SW5 SW_Push, SW6 SW_Push, SW7 SW_Push, SW8 SW_Push, SW9 SW_Push, U1 STM32G0B1RETx, U2 LD1117S33TR_SOT223

Commit message: deck_v3: Tweak schematic layout for improved visibility of components.
No electrical change.

Signed-off-by: Damien George <dpgeorge@georgerobotics.com.au>
Parts:
- J11: value DNP -> CONN_A_AUX
Changed lines of the file:
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@@
 			)
 		)
-		(property "Value" "DNP"
+		(property "Value" "CONN_A_AUX"
 			(at 0 -7.46 0)
 			(layer "B.Fab")
